File: ESP TEmperature Sensor/ESP01Temperature.sch (KiCad schematic (older format))
At the start: 10 parts, among them K1 CONN_3, P1 CONN_4X2, P2 CONN_2, SW1 PROG, SW2 RESET, U1 DS18B20

Commit message: PCB Design
Kicad design files for build PCB
Parts:
- removed P1: CONN_4X2, Pin_Headers:Pin_Header_Straight_2x04, symbol CONN_4X2
- added C1, C2: 33u, Capacitors_SMD:C_1206_HandSoldering, symbol C
- added P1: CONN_6, Connectors_Molex:Molex_KK-6410-06_06x2.54mm_Straight, symbol CONN_6
- added Q1: MCP1700T-3302E/TT, TO_SOT_Packages_SMD:SOT-23, symbol MCP1700T-3302E/TT
- added U2: ESP-01v090, ESP8266:ESP-01, symbol ESP-01v090
- K1: value CONN_3 -> CONN_5; footprint Pin_Headers:Pin_Header_Angled_1x03 -> Connectors_Molex:Molex_KK-6410-05_05x2.54mm_Straight; symbol CONN_3 -> CONN_5
- R1, R2, R3, R4: footprint Discret:R3 -> Resistors_SMD:R_1206_HandSoldering
- U1: footprint Pin_Headers:Pin_Header_Angled_1x03 -> TO_SOT_Packages_THT:TO-92_Molded_Narrow
Connections:
- net GND: now also C1.2, C2.1, Q1.1 (GND), U2.2 (GND)
- net GPIO0: now also K1.4, U2.6 (GPIO0)
- net GPIO2: now also K1.5, U2.4 (GPIO2)
- net RX: now also U2.8 (URXD)
- net TX: now also U2.1 (UTXD)
- net VDD: now also C2.2, Q1.2 (Vout), U2.3 (CH_PD), U2.7 (VCC); no longer P2.2 (PM)
- net RESET: no longer names the net of R4.2, SW2.1
- net RESET: now also U2.5 (RST)
- new net: C1.1, P2.2 (PM), Q1.3 (Vin)
Other:
- moved on the sheet: P2, R1, R2, R3, R4, SW1, SW2, U1

Commit message: Changes to who knows what.
Uncommitted changes to stuff. Tidying up…
Parts:
- Q1: symbol MCP1700T-3302E/TT -> MCP1700T-3302E/TT-RESCUE-ESP01Temperature
Changed lines of the file:
@@
 EESchema Schematic File Version 2
+LIBS:ESP01Temperature-rescue
 LIBS:power
 LIBS:device
@@
 	4350 3700 4350 3550
 Wire Wire Line
-	5200 3200 5200 3550
-Wire Wire Line
-	5200 3550 5200 4250
+	5200 3200 5200 4250
 Connection ~ 5200 3550
 Wire Wire Line
-	5200 2700 5600 2700
-Wire Wire Line
-	5600 2700 7200 2700
-Wire Wire Line
-	7200 2700 7300 2700
-Wire Wire Line
-	7300 2700 7950 2700
-Wire Wire Line
-	7950 2700 8400 2700
+	5200 2700 8400 2700
 Connection ~ 5600 2700
 $Comp
@@
 $EndComp
 Wire Wire Line
-	1900 3250 1900 3450
-Wire Wire Line
-	1900 3450 1900 3650
+	1900 3250 1900 3650
 $Comp
 L R R1
@@
 	2350 3950 2350 4150
 Wire Wire Line
-	2300 4150 2350 4150
-Wire Wire Line
-	2350 4150 3200 4150
+	2300 4150 3200 4150
 Wire Wire Line
 	1900 4550 1900 4800
@@
 $EndComp
 $Comp
-L MCP1700T-3302E/TT Q1
+L MCP1700T-3302E/TT-RESCUE-ESP01Temperature Q1
 U 1 1 5807E986
 P 3550 1300
@@
 $EndComp
 Wire Wire Line
-	2100 1300 2600 1300
-Wire Wire Line
-	2600 1300 2950 1300
+	2100 1300 2950 1300
 Wire Wire Line
 	3550 800  3550 750
@@
 $EndComp
 Wire Wire Line
-	7600 4250 8450 4250
-Wire Wire Line
-	8450 4250 8500 4250
+	7600 4250 8500 4250
 Wire Wire Line
 	7600 4150 7950 4150
 Wire Wire Line
-	7950 2700 7950 4150
-Wire Wire Line
-	7950 4150 7950 4350
+	7950 2700 7950 4350
 Wire Wire Line
 	7950 4350 7600 4350
@@
 RX
 Wire Wire Line
-	3200 4350 5600 4350
-Wire Wire Line
-	5600 4350 5700 4350
+	3200 4350 5700 4350
 Wire Wire Line
 	5200 4250 5700 4250
